File: car-shield.kicad_pcb (KiCad board)
At the start: 2 copper layers, 66.7 x 64.1 mm, 34 parts

Commit message: updated resistor parts and Freepik notice
Other:
- board text added: "car designed by Freepik"
Changed lines of the file:
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@@
   )
   (gr_rect (start 106.68 66.04) (end 173.355 130.175) (layer "Edge.Cuts") (width 0.1) (fill none))
+  (gr_text "car designed by Freepik" (at 165.1 104.14 90) (layer "F.Paste")
+    (effects (font (size 1 1) (thickness 0.15)))
+  )
 )

Commit message: updated car footprint
Parts:
- added REF**: car, car:car, F.Cu at (145.3, 77.8)
- moved Ref** 34.9 mm to (78.7, 97.8)
- moved D7 4.93 mm to (154.9, 100.3)

Commit message: some initial routing
Parts:
- added BZ1: Buzzer, Buzzer_Beeper:Buzzer_15x7.5RM7.6, B.Cu at (159.1, 99.1)
- moved D8 3.47 mm to (161.7, 116.7), turned to 30 degrees
- moved D9 3.17 mm to (149.0, 116.7), turned to 150 degrees
- moved D4 2.98 mm to (161.9, 80.9), turned to -40 degrees
- moved D1 2.64 mm to (151.4, 79.1), turned to -165 degrees
- moved D3 2.56 mm to (148.7, 80.9), turned to -140 degrees
- moved D2 2.29 mm to (159.3, 79.1), turned to -15 degrees
- moved D6 2.25 mm to (164.7, 91.2), turned to -20 degrees
- moved D5 1.82 mm to (145.9, 91.2), turned to -160 degrees
- moved R10 0.38 mm to (140.7, 76.1)
- moved D7 0.38 mm to (155.3, 100.3)
- moved R7 0.25 mm to (135.6, 76.1)
Routing:
- net GND: track 0.00 -> 236.9 mm, vias 0 -> 15
- net VDD: track 0.00 -> 103.5 mm, vias 0 -> 7
- net Net-(D8-Pad2): track 0.00 -> 64.7 mm, vias 0 -> 2
- net speed_indicator: track 0.00 -> 63.2 mm
- net sw_right: track 0.00 -> 61.3 mm, vias 0 -> 2
- net sw_stop: track 0.00 -> 56.2 mm, vias 0 -> 2
- net sw_accel: track 0.00 -> 53.2 mm, vias 0 -> 2
- net Net-(D9-Pad2): track 0.00 -> 42.5 mm, vias 0 -> 2
- net Net-(D7-Pad2): track 0.00 -> 40.0 mm, vias 0 -> 5
- net sw_left: track 0.00 -> 37.1 mm, vias 0 -> 1
- net sw_high_b: track 0.00 -> 36.7 mm, vias 0 -> 2
- net sw_decel: track 0.00 -> 36.1 mm, vias 0 -> 2
- net Net-(D6-Pad2): track 0.00 -> 29.3 mm, vias 0 -> 2
- net sw_dipped_b: track 0.00 -> 23.0 mm, vias 0 -> 2
- net Net-(D5-Pad2): track 0.00 -> 17.7 mm, vias 0 -> 2
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- added copper zone on B.Cu, net GND
- added copper zone on F.Cu, net GND
Other:
- board size 66.7 x 64.1 mm -> 47.1 x 53.6 mm

Commit message: layout tweaks
Parts:
- removed Ref**: Val**, HTL Weiz Logo:logo
- SW_accel1, SW_decel1, SW_dipped_b1, SW_high_b1, SW_left1, SW_right1, SW_stop1: footprint Button_Switch_SMD:SW_SPST_SKQG_WithoutStem -> car:SW_SPST_TS-1187A
- moved BZ1 27.2 mm to (135.4, 85.7)
- moved SW_decel1 6.30 mm to (126.4, 110.5)
- moved SW_dipped_b1 6.30 mm to (136.6, 110.5)
- moved SW_accel1 4.59 mm to (126.4, 100.2)
- moved SW_high_b1 4.59 mm to (136.6, 100.2)
- moved R7 3.81 mm to (131.8, 76.1)
- moved SW_left1 3.45 mm to (126.4, 81.6)
- moved SW_right1 3.45 mm to (136.6, 81.6)
- moved SW_stop1 2.30 mm to (131.5, 89.8)
Routing:
- net speed_indicator: track 63.2 -> 17.1 mm, vias 0 -> 1
- net sw_dipped_b: track 23.0 -> 29.3 mm
- net Net-(D7-Pad2): track 40.0 -> 44.8 mm
- net sw_high_b: track 36.7 -> 41.0 mm
- net sw_right: track 61.3 -> 64.7 mm
- net sw_accel: track 53.2 -> 56.5 mm
- net sw_decel: track 36.1 -> 39.2 mm
- net sw_left: track 37.1 -> 34.1 mm
- net VDD: track 103.5 -> 101.1 mm
- net sw_stop: track 56.2 -> 58.5 mm
- net GND: track 236.9 -> 234.8 mm
Other:
- outline, holes or cut-outs redrawn
- board text added: "PCB: wu@htlweiz.at"

Commit message: final touches for revA
Other:
- board text added: "github.com/htlweiz/car-shield"
- board text added: "revA"

Commit message: rev0
Parts:
- added REF**: logo-6mm, HTL Weiz Logo:logo-6mm, F.Cu at (129.6, 114.2)
- added REF**: logo-6mm, HTL Weiz Logo:logo-6mm, B.Cu at (161.6, 87.4)
Routing:
- net GND: track 234.8 -> 235.5 mm
Other:
- board text added: "rev0"
- board text removed: "revA"
