File: car-shield.kicad_sch (KiCad schematic)
At the start: 33 parts

Commit message: updated resistor parts and Freepik notice
Parts:
- R10, R11, R12, R13, R14, R15, R16: LCSC C11616 -> C25744
Changed lines of the file:
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@@
       (effects (font (size 1.27 1.27)) hide)
     )
-    (property "LCSC" "C11616" (id 4) (at 45.72 33.0199 0)
+    (property "LCSC" "C25744" (id 4) (at 45.72 33.0199 0)
       (effects (font (size 1.27 1.27)) hide)
     )
@@
       (effects (font (size 1.27 1.27)) hide)
     )
-    (property "LCSC" "C11616" (id 4) (at 45.72 111.7599 0)
+    (property "LCSC" "C25744" (id 4) (at 45.72 111.7599 0)
       (effects (font (size 1.27 1.27)) hide)
     )
@@
       (effects (font (size 1.27 1.27)) hide)
     )
-    (property "LCSC" "C11616" (id 4) (at 63.5 33.0199 0)
+    (property "LCSC" "C25744" (id 4) (at 63.5 33.0199 0)
       (effects (font (size 1.27 1.27)) hide)
     )
@@
       (effects (font (size 1.27 1.27)) hide)
     )
-    (property "LCSC" "C11616" (id 4) (at 45.72 72.3899 0)
+    (property "LCSC" "C25744" (id 4) (at 45.72 72.3899 0)
       (effects (font (size 1.27 1.27)) hide)
     )
@@
       (effects (font (size 1.27 1.27)) hide)
     )
-    (property "LCSC" "C11616" (id 4) (at 27.94 72.3899 0)
+    (property "LCSC" "C25744" (id 4) (at 27.94 72.3899 0)
       (effects (font (size 1.27 1.27)) hide)
     )
@@
       (effects (font (size 1.27 1.27)) hide)
     )
-    (property "LCSC" "C11616" (id 4) (at 27.94 111.7599 0)
+    (property "LCSC" "C25744" (id 4) (at 27.94 111.7599 0)
       (effects (font (size 1.27 1.27)) hide)
     )
@@
       (effects (font (size 1.27 1.27)) hide)
     )
-    (property "LCSC" "C11616" (id 4) (at 27.94 33.0199 0)
-      (effects (font (size 1.27 1.27)) hide)
-    )
+    (property "LCSC" "C25744" (id 4) (at 27.94 33.0199 0)
+      (effects (font (size 1.27 1.27)) hide)
+    )

Commit message: some initial routing
Parts:
- added BZ1: Buzzer, Buzzer_Beeper:Buzzer_15x7.5RM7.6, symbol Device:Buzzer
Connections:
- net GND: now also BZ1.2 (+)
- net speed_indicator: now also BZ1.1 (-)
Changed lines of the file:
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@@
+    )
+  )
+  (global_label "speed_indicator" (shape input) (at 205.74 140.97 180) (fields_autoplaced)
+    (effects (font (size 1.27 1.27)) (justify right))
+    (property "Intersheet References" "${INTERSHEET_REFS}" (id 0) (at 188.4498 140.8906 0)
+      (effects (font (size 1.27 1.27)) (justify right) hide)
     )
   )
@@
     (pin "1")
   )
+  (symbol (lib_id "Device:Buzzer") (at 208.28 143.51 0) (unit 1)
+    (in_bom yes) (on_board yes) (fields_autoplaced)
+    (property "Reference" "BZ1" (id 0) (at 212.09 142.2399 0)
+      (effects (font (size 1.27 1.27)) (justify left))
+    )
+    (property "Value" "Buzzer" (id 1) (at 212.09 144.7799 0)
+      (effects (font (size 1.27 1.27)) (justify left))
+    )
+    (property "Footprint" "Buzzer_Beeper:Buzzer_15x7.5RM7.6" (id 2) (at 207.645 140.97 90)
+      (effects (font (size 1.27 1.27)) hide)
+    )
+    (property "Datasheet" "~" (id 3) (at 207.645 140.97 90)
+      (effects (font (size 1.27 1.27)) hide)
+    )
+    (pin "1")
+    (pin "2")
+  )
   (symbol (lib_id "Switch:SW_SPST") (at 60.96 44.45 90) (unit 1)
     (in_bom yes) (on_board yes) (fields_autoplaced)
@@
     (pin "1")
     (pin "2")
+  )
+  (symbol (lib_id "power:GND") (at 205.74 146.05 0) (unit 1)
+    (in_bom yes) (on_board yes) (fields_autoplaced)
+    (property "Reference" "#PWR0115" (id 0) (at 205.74 152.4 0)
+      (effects (font (size 1.27 1.27)) hide)
+    )
+    (property "Value" "GND" (id 1) (at 205.74 151.13 0))
+    (property "Footprint" "" (id 2) (at 205.74 146.05 0)
+      (effects (font (size 1.27 1.27)) hide)
+    )
+    (property "Datasheet" "" (id 3) (at 205.74 146.05 0)
+      (effects (font (size 1.27 1.27)) hide)
+    )
+    (pin "1")
   )
   (symbol (lib_id "Switch:SW_SPST") (at 25.4 123.19 90) (unit 1)
@@
       (reference "#PWR0114") (unit 1) (value "VDD") (footprint "")
     )
+    (path "/a42257f5-cf71-4f1d-a169-14d91afdc944"
+      (reference "#PWR0115") (unit 1) (value "GND") (footprint "")
+    )
     (path "/f264adcd-006b-4f60-a0e5-5dc1e994d3db"
       (reference "A1") (unit 1) (value "Arduino_UNO_R2") (footprint "Module:Arduino_UNO_R2")
     )
+    (path "/653ad176-25a1-4164-916e-024925232301"
+      (reference "BZ1") (unit 1) (value "Buzzer") (footprint "Buzzer_Beeper:Buzzer_15x7.5RM7.6")
+    )
     (path "/96a8adfc-6509-4e50-b0de-151a609e8367"

Commit message: rev0
Other:
- company: (none) -> HTL Weiz
- title: (none) -> CAR SHIELD
- moved on the sheet: A1, BZ1, D1, D2, D3, D4, D5, D6, D7, D8, D9, R1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
